File: circuit/pi-pico-alarmclock/pi-pico-alarmclock.kicad_sch (KiCad schematic)
At the start: 33 parts, among them J1 Screw_Terminal_2_P5.00mm, J2 BTN GREEN, J3 BTN BLUE, J4 BTN_YELLOW, J5 NEOPIXEL, J6 OLED, J7 BAT - Screw_Terminal_2_P5.00mm, Q1 IRLZ44N, Q3 IRF9540, Q4 IRLZ44N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

Commit message: Add TP4056 charger footprint and fix orientations
Parts:
- U3: footprint (none) -> common-hobby-things:TP4056_charger_board
Connections:
- net GND: now also U3.2 (DC-); no longer U3.6 (OUT-)
- net VBUS: now also U3.1 (DC+); no longer U3.3 (DC+)
- net at J7.1 (BAT+): now also U3.5 (BAT+); no longer U3.1 (BAT+)
- net at J7.2 (BAT-): now also U3.6 (BAT-); no longer U3.2 (BAT-)
- net at Q3.2 (D): now also U3.3 (OUT+); no longer U3.5 (OUT+)
Changed lines of the file:
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@@
 			)
 		)
-		(property "Footprint" ""
+		(property "Footprint" "common-hobby-things:TP4056_charger_board"
 			(at 160.02 50.8 0)
 			(effects

Commit message: First Layout draft, no tracks yet
Connections:
- net GP28: now also U1.34 (GPIO28_ADC2)
- net VBUS: no longer U1.34 (GPIO28_ADC2)
- net BAT+: now reaches J7.1 (BAT+), U3.5 (BAT+)
- net BAT-: now reaches J7.2 (BAT-), U3.6 (BAT-)
Changed lines of the file:
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@@
+		)
+	)
+	(label "BAT-"
+		(at 173.99 48.26 0)
+		(effects
+			(font
+				(size 1.27 1.27)
+			)
+			(justify left bottom)
 		)
 	)
@@
 		)
 	)
+	(label "BAT+"
+		(at 144.78 48.26 0)
+		(effects
+			(font
+				(size 1.27 1.27)
+			)
+			(justify left bottom)
+		)
+	)
 	(label "GP22"
 		(at 144.78 146.05 0)
@@
 	(label "GP27"
 		(at 107.95 68.58 0)
+		(effects
+			(font
+				(size 1.27 1.27)
+			)
+			(justify left bottom)
+		)
+	)
+	(label "GP28"
+		(at 107.95 63.5 0)
 		(effects
 			(font
@@
 		(effects
 			(font
-				(size 1.27 1.27)
-			)
-			(justify left bottom)
-		)
-	)
-	(label "VBUS"
-		(at 107.95 63.5 0)
-		(effects
-			(font
