File: circuit/pi-pico-alarmclock/pi-pico-alarmclock.kicad_sch (KiCad schematic)
At the start: 33 parts, among them J1 Screw_Terminal_2_P5.00mm, J2 BTN GREEN, J3 BTN BLUE, J4 BTN_YELLOW, J5 NEOPIXEL, J6 OLED, J7 BAT - Screw_Terminal_2_P5.00mm, Q1 IRLZ44N, Q3 IRF9540, Q4 IRLZ44N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

Commit message: pcb and schemativ v0.2: Fix ground bounce by providing direct path to battery ground
Connections:
- net BAT- is gone; now on net GND: J7.2 (BAT-), U3.6 (BAT-)
Other:
- company: (none) -> rafael
- title: (none) -> pi-pico-alarmclock-rust
Changed lines of the file:
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@@
 	(generator_version "9.0")
 	(paper "A4")
+	(title_block
+		(title "pi-pico-alarmclock-rust")
+		(date "2025-11-20")
+		(rev "v0.2")
+		(company "rafael")
+	)
 	(rectangle
 		(start 179.07 111.76)
@@
 	)
 	(junction
+		(at 161.29 44.45)
+		(diameter 0)
+		(color 0 0 0 0)
+	)
+	(junction
 		(at 153.67 97.79)
 		(diameter 0)
@@
 	)
 	(symbol
+		(lib_id "power:GND")
+		(at 161.29 44.45 0)
+		(unit 1)
+		(exclude_from_sim no)
+		(in_bom yes)
+		(on_board yes)
+		(dnp no)
+		(property "Reference" "#PWR03"
+			(at 161.29 50.8 0)
+			(effects
+				(font
+					(size 1.27 1.27)
+				)
+				(hide yes)
+			)
+		)
+		(property "Value" "GND"
+			(at 164.084 46.99 0)
+			(effects
+				(font
+					(size 1.27 1.27)
+				)
+			)
+		)
+		(property "Footprint" ""
+			(at 161.29 44.45 0)
+			(effects
+				(font
+					(size 1.27 1.27)
+				)
+				(hide yes)
+			)
+		)
+		(property "Datasheet" ""
+			(at 161.29 44.45 0)
+			(effects
+				(font
+					(size 1.27 1.27)
+				)
+				(hide yes)
+			)
+		)
+		(property "Description" "Power symbol creates a global label with name \"GND\" , ground"
+			(at 161.29 44.45 0)
+			(effects
+				(font
+					(size 1.27 1.27)
+				)
+				(hide yes)
+			)
+		)
+		(pin "1"
+		)
+		(instances
+			(project "pi-pico-alarmclock"
+				(path "/4c5cb0eb-2550-406b-8a38-335faa16f981"
+					(reference "#PWR03")
+					(unit 1)
+				)
+			)
+		)
+	)
+	(symbol
 		(lib_id "PCM_SL_Screw_Terminal:Screw_Terminal_2_P5.00mm")
 		(at 195.58 147.32 180)
@@
 		(dnp no)
 		(property "Reference" "U3"
-			(at 160.274 48.514 0)
+			(at 159.258 48.768 0)
 			(effects
 				(font
